File: Kicad/neotron-pico-btx.kicad_pcb (KiCad board)
At the start: 4 copper layers, 243.8 x 171.4 mm, 242 parts, among them J1001 Conn_01x05, J1002 Conn_01x02, J1003 Conn_01x02, J1004 Conn_01x02, J1005 Conn_01x02, J1006 Conn_01x04, J1007 Double-mini-DIN-6, J1101 SD_Card, J1301 Jack 2.1mm 6.3mm, J1302 Conn_02x02S, J1303 Conn_01x04S, J401 DE15HD, J801 Conn_01x04, J802 Conn_02x05, J803 Conn_01x04, J901 Conn_01x06, J902 Neotron-Expansion-Slot, J903 Neotron-Expansion-Slot, J904 Neotron-Expansion-Slot, J905 Neotron-Expansion-Slot, J906 Conn_01x09, J907 Conn_01x09, J908 Conn_01x09, Q1001 2N7002, Q1002 2N7002, Q1003 SS8050, Q1301 AO3401A, Q1302 SS8550, Q1303 SS8050, Q201 DMG2305UX, SW1001 SW_Push, SW1002 SW_Push, U1001 STM32F030K6T6, U1201 DS1307Z+, U1301 DC-DC Module, U1302 AMS1117-3.3, U1303 HT75xx-1-SOT89, U201 Pico, U301 MCP23S17_SO, U302 74HC138, U303 74AHC1G04, U401 THS7316, U402 TPD7S019, U801 TLV320AIC23BPW, U802 STX-4335-5BGP-S1, Y1201 32,768 Hz, Y801 12M 20pF

Commit message: - Enhance conversion report with comprehensive details
Co-Authored-By: Erkin Alp Güney <erkinalp9035@gmail.com>
Parts:
- D1001, D1002, D301, D302, D303, D304: moved to B.Cu
- moved C1303 264.3 mm to (-0.16, 173.7)
- moved J1001 264.3 mm to (-0.16, 76.8)
- moved J901 264.3 mm to (-0.16, 95.2)
- moved U1301 263.0 mm to (0.47, 154.3)
- moved H103 261.8 mm to (1.11, 58.4)
- moved H107 261.8 mm to (1.11, 190.5)
- moved R1014 261.8 mm to (1.11, 47.6)
- moved L1301 258.0 mm to (3.02, 120.1)
- moved R1016 256.7 mm to (3.65, 47.6)
- moved J1007 255.5 mm to (4.25, 36.5)
- moved C1301 254.2 mm to (4.92, 112.4)
- moved C1302 254.2 mm to (4.92, 132.7)
- moved TP1301 252.3 mm to (5.87, 116.8)
- moved R1015 251.6 mm to (6.19, 47.6)
- moved JP1001 249.1 mm to (7.46, 67.6)
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Routing:
- net GND: track 148.4 -> 757.0 mm, vias 223 -> 218
- net /Audio/3V3_DIGITAL: track 14.6 -> 231.2 mm, vias 0 -> 1
- net /Slots and Peripherals/BMC/~{BUTTON_PWR}: track 205.7 -> 0.00 mm, vias 2 -> 0
- net /Slots and Peripherals/PICO_SDA: track 307.9 -> 128.9 mm, vias 1 -> 2
- net /Slots and Peripherals/BMC/BUZZER: track 143.4 -> 0.00 mm
- net unconnected-(U801-CLKOUT-Pad2): track 0.00 -> 120.9 mm, vias 0 -> 1
- net /Audio/AUDIO_ADC_DATA: track 120.9 -> 0.00 mm, vias 1 -> 0
- net /Slots and Peripherals/BMC_SCL: track 102.4 -> 0.00 mm, vias 3 -> 0
- net /IO Expander/HDD_LED: track 58.9 -> 0.00 mm
- net /Audio/MicBias: track 46.0 -> 0.00 mm, vias 2 -> 0
- net Net-(U801-~{CS}): track 8.07 -> 54.1 mm, vias 0 -> 2
- net Net-(U801-MODE): track 6.99 -> 45.6 mm, vias 0 -> 3
- net /Audio/MicIn: track 37.4 -> 1.22 mm, vias 2 -> 1
- net /Audio/RLineIn: track 37.5 -> 1.71 mm, vias 2 -> 1
- net Net-(J1005-Pin_2): track 29.6 -> 0.00 mm
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Other:
- board size 243.8 x 171.4 mm -> 922.5 x 1138.1 mm
- board text added: "Neotron Pico: ${version}"
- board text removed: "Neotron Pico: 1.0-BTX"

Commit message: - Ensure compatibility with BTX cases
Co-Authored-By: Erkin Alp Güney <erkinalp9035@gmail.com>
Parts:
- H101, H102, H103, H104, H105, H106, H107: value MountingHole_Pad -> MountingHole; footprint MountingHole:MountingHole_4.3mm_M4_Pad_Via -> (none)
- moved H102 271.7 mm to (6.35, 260.6)
- moved H103 261.8 mm to (257.6, 6.35)
- moved H101 200.1 mm to (6.35, 6.35)
- moved H105 197.8 mm to (132.0, 6.35)
- moved H107 142.8 mm to (132.0, 133.5)
- moved H104 77.5 mm to (257.6, 260.6)
- moved H106 75.0 mm to (132.0, 260.6)
Connections:
- H101 pad 1: GND -> (no net)
- H102 pad 1: GND -> (no net)
- H103 pad 1: GND -> (no net)
- H104 pad 1: GND -> (no net)
- H105 pad 1: GND -> (no net)
- H106 pad 1: GND -> (no net)
- H107 pad 1: GND -> (no net)
Routing:
- net /VGA_HSYNC: track 45.2 -> 0.00 mm
- net /Slots and Peripherals/SPI_CIPO: track 353.4 -> 398.6 mm
Other:
- board size 922.5 x 1138.1 mm -> 243.8 x 171.5 mm
