File: Kicad/neotron-pico-btx.kicad_pcb (KiCad board)
At the start: 4 copper layers, 243.8 x 171.5 mm, 242 parts, among them J1001 Conn_01x05, J1002 Conn_01x02, J1003 Conn_01x02, J1004 Conn_01x02, J1005 Conn_01x02, J1006 Conn_01x04, J1007 Double-mini-DIN-6, J1101 SD_Card, J1301 Jack 2.1mm 6.3mm, J1302 Conn_02x02S, J1303 Conn_01x04S, J401 DE15HD, J801 Conn_01x04, J802 Conn_02x05, J803 Conn_01x04, J901 Conn_01x06, J902 Neotron-Expansion-Slot, J903 Neotron-Expansion-Slot, J904 Neotron-Expansion-Slot, J905 Neotron-Expansion-Slot, J906 Conn_01x09, J907 Conn_01x09, J908 Conn_01x09, Q1001 2N7002, Q1002 2N7002, Q1003 SS8050, Q1301 AO3401A, Q1302 SS8550, Q1303 SS8050, Q201 DMG2305UX, SW1001 SW_Push, SW1002 SW_Push, U1001 STM32F030K6T6, U1201 DS1307Z+, U1301 DC-DC Module, U1302 AMS1117-3.3, U1303 HT75xx-1-SOT89, U201 Pico, U301 MCP23S17_SO, U302 74HC138, U303 74AHC1G04, U401 THS7316, U402 TPD7S019, U801 TLV320AIC23BPW, U802 STX-4335-5BGP-S1, Y1201 32,768 Hz, Y801 12M 20pF

Commit message: Complete microBTX conversion with proper board dimensions and mounting holes
Co-Authored-By: Erkin Alp Güney <erkinalp9035@gmail.com>
Parts:
- removed H101, H102, H103, H104, H105, H106, H107: MountingHole, 
- added H1: MountingHole_3.2mm_M3, MountingHole_3.2mm_M3, F.Cu at (6.35, 6.35)
- added H2: MountingHole_3.2mm_M3, MountingHole_3.2mm_M3, F.Cu at (6.35, 260.6)
- added H3: MountingHole_3.2mm_M3, MountingHole_3.2mm_M3, F.Cu at (257.6, 6.35)
- added H4: MountingHole_3.2mm_M3, MountingHole_3.2mm_M3, F.Cu at (257.6, 260.6)
- added H5: MountingHole_3.2mm_M3, MountingHole_3.2mm_M3, F.Cu at (130.0, 133.5)
Other:
- board size 243.8 x 171.5 mm -> 264 x 267 mm

Commit message: Add SRM mounting hole position verification and region analysis
Co-Authored-By: Erkin Alp Güney <erkinalp9035@gmail.com>
Parts:
- added HSRM1: MountingHole_3.2mm_M3, MountingHole_3.2mm_M3, F.Cu at (115.0, 118.5)
- added HSRM2: MountingHole_3.2mm_M3, MountingHole_3.2mm_M3, F.Cu at (115.0, 148.5)
- added HSRM3: MountingHole_3.2mm_M3, MountingHole_3.2mm_M3, F.Cu at (145.0, 118.5)
- added HSRM4: MountingHole_3.2mm_M3, MountingHole_3.2mm_M3, F.Cu at (145.0, 148.5)
