File: Kicad/neotron-pico-btx.kicad_pcb (KiCad board)
At the start: 4 copper layers, 264 x 267 mm, 244 parts, among them J1001 Conn_01x05, J1002 Conn_01x02, J1003 Conn_01x02, J1004 Conn_01x02, J1005 Conn_01x02, J1006 Conn_01x04, J1007 Double-mini-DIN-6, J1101 SD_Card, J1301 Jack 2.1mm 6.3mm, J1302 Conn_02x02S, J1303 Conn_01x04S, J401 DE15HD, J801 Conn_01x04, J802 Conn_02x05, J803 Conn_01x04, J901 Conn_01x06, J902 Neotron-Expansion-Slot, J903 Neotron-Expansion-Slot, J904 Neotron-Expansion-Slot, J905 Neotron-Expansion-Slot, J906 Conn_01x09, J907 Conn_01x09, J908 Conn_01x09, Q1001 2N7002, Q1002 2N7002, Q1003 SS8050, Q1301 AO3401A, Q1302 SS8550, Q1303 SS8050, Q201 DMG2305UX, SW1001 SW_Push, SW1002 SW_Push, U1001 STM32F030K6T6, U1201 DS1307Z+, U1301 DC-DC Module, U1302 AMS1117-3.3, U1303 HT75xx-1-SOT89, U201 Pico, U301 MCP23S17_SO, U302 74HC138, U303 74AHC1G04, U401 THS7316, U402 TPD7S019, U801 TLV320AIC23BPW, U802 STX-4335-5BGP-S1, Y1201 32,768 Hz, Y801 12M 20pF

Commit message: Complete BTX conversion with SRM mounting holes and verification
Co-Authored-By: Erkin Alp Güney <erkinalp9035@gmail.com>
Parts:
- added H10: MOUNT_HOLE_SRM, , F.Cu at (190.0, 130.0)
- added H11: MOUNT_HOLE_SRM, , F.Cu at (190.0, 230.0)
- added H12: MOUNT_HOLE_SRM, , F.Cu at (250.0, 130.0)
- added H13: MOUNT_HOLE_SRM, , F.Cu at (250.0, 230.0)
- moved U1301 133.2 mm to (132.0, 133.5)
- moved U1001 127.6 mm to (132.0, 133.5)
- moved U201 121.9 mm to (132.0, 133.5)
- moved U1303 114.8 mm to (132.0, 133.5)
- moved U1302 104.1 mm to (132.0, 133.5)
- moved U402 103.6 mm to (132.0, 133.5)
- moved U802 99.3 mm to (132.0, 133.5)
- moved U401 91.4 mm to (132.0, 133.5)
- moved U303 71.7 mm to (132.0, 133.5)
- moved U302 68.3 mm to (132.0, 133.5)
- moved U301 56.5 mm to (132.0, 133.5)
- moved U801 45.2 mm to (132.0, 133.5)
- moved J1007 8.95 mm to (13.2, 36.5)
- moved C1303 7.02 mm to (6.86, 173.7)
- moved L1301 6.96 mm to (9.97, 120.1)
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Routing:
- net GND: track 757.0 -> 18189.8 mm, vias 218 -> 0
- net +3V3: track 43.7 -> 3774.2 mm, vias 38 -> 0
- net +5V: track 822.7 -> 4189.2 mm, vias 15 -> 0
- net /Slots and Peripherals/SPI_CIPO: track 398.6 -> 1710.9 mm, vias 5 -> 0
- net /Slots and Peripherals/PICO_SDA: track 128.9 -> 746.1 mm, vias 2 -> 0
- net VDC: track 69.6 -> 560.9 mm
- net /Slots and Peripherals/PICO_SCL: track 304.5 -> 764.1 mm, vias 1 -> 0
- net +3.3VP: track 125.0 -> 581.8 mm, vias 3 -> 0
- net /Slots and Peripherals/SPI_COPI: track 350.6 -> 769.2 mm, vias 3 -> 0
- net /Slots and Peripherals/SPI_CLK: track 341.1 -> 753.1 mm, vias 3 -> 0
- net /Slots and Peripherals/~{RESET}: track 415.2 -> 687.1 mm, vias 5 -> 0
- net /Slots and Peripherals/BMC/PS2_CLK1: track 35.7 -> 303.2 mm, vias 2 -> 0
- net /Slots and Peripherals/BMC/PS2_CLK0: track 40.8 -> 306.5 mm
- net /Slots and Peripherals/BMC/PS2_DAT1: track 40.4 -> 302.4 mm, vias 2 -> 0
- net /Slots and Peripherals/BMC/PS2_DAT0: track 48.7 -> 310.1 mm, vias 2 -> 0
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